Commit message: Create roburoc_description package for robot model separation

File: src/roburoc_description/urdf/RobuROC_core.urdf.xacro (robot description, xacro)
@@ -26,5 +26,5 @@
             <origin xyz="${chassis_vis_origin}" rpy="${rot_90} 0 ${rot_90}"/>
             <geometry>
-                <mesh filename="file://$(find roburoc_sim)/meshes/chassis.STL" scale="${scale}"/>
+                <mesh filename="file://$(find roburoc_description)/meshes/chassis.STL" scale="${scale}"/>
             </geometry>
             <material name="grey" />
@@ -55,5 +55,5 @@
             <origin xyz="0 0 0" rpy="0 ${rot_90} 0"/>
             <geometry>
-                <mesh filename="file://$(find roburoc_sim)/meshes/wheel.STL" scale = "${scale}"/>
+                <mesh filename="file://$(find roburoc_description)/meshes/wheel.STL" scale = "${scale}"/>
             </geometry>
             <material name="black" />
@@ -84,5 +84,5 @@
             <origin xyz="0 0 0" rpy="0 ${rot_90} 0"/>
             <geometry>
-                <mesh filename="file://$(find roburoc_sim)/meshes/wheel.STL" scale = "${scale}"/>
+                <mesh filename="file://$(find roburoc_description)/meshes/wheel.STL" scale = "${scale}"/>
             </geometry>
             <material name="black" />
@@ -113,5 +113,5 @@
             <origin xyz="0 0 0" rpy="0 ${rot_90} 0"/>
             <geometry>
-                <mesh filename="file://$(find roburoc_sim)/meshes/wheel.STL" scale = "${scale}"/>
+                <mesh filename="file://$(find roburoc_description)/meshes/wheel.STL" scale = "${scale}"/>
             </geometry>
             <material name="black" />
@@ -142,5 +142,5 @@
             <origin xyz="0 0 0" rpy="0 ${rot_90} 0"/>
             <geometry>
-                <mesh filename="file://$(find roburoc_sim)/meshes/wheel.STL" scale = "${scale}"/>
+                <mesh filename="file://$(find roburoc_description)/meshes/wheel.STL" scale = "${scale}"/>
             </geometry>
             <material name="black" />

File: src/roburoc_description/urdf/VLP-16.urdf.xacro (robot description, xacro)
@@ -17,10 +17,10 @@
       <visual>
         <geometry>
-          <mesh filename="file://$(find roburoc_sim)/meshes/VLP16_base_1.dae"/>
+          <mesh filename="file://$(find roburoc_description)/meshes/VLP16_base_1.dae"/>
         </geometry>
       </visual>
       <visual>
         <geometry>
-          <mesh filename="file://$(find roburoc_sim)/meshes/VLP16_base_2.dae"/>
+          <mesh filename="file://$(find roburoc_description)/meshes/VLP16_base_2.dae"/>
         </geometry>
       </visual>
@@ -46,5 +46,5 @@
         <origin xyz="0 0 -0.0377"/>
         <geometry>
-          <mesh filename="file://$(find roburoc_sim)/meshes/VLP16_scan.dae"/>
+          <mesh filename="file://$(find roburoc_description)/meshes/VLP16_scan.dae"/>
         </geometry>
       </visual>
