Commit message: Migrate to Gazebo Harmonic: Update URDF models, launch files, and dependencies for improved simulation support

File: src/roburoc_description/urdf/RobuROC_gazebo_sim.xacro (robot description, xacro)
@@ -1,40 +1,82 @@
 <?xml version="1.0"?>
 <robot xmlns:xacro="http://www.ros.org/wiki/xacro">
-    <!-- This is RobuROC model for gazebo simulation -->
+    <!-- This is RobuROC model for Gazebo Harmonic simulation -->
     <!-- Model visualisation and collision is made of simple shapes box and cylinders-->
-    <!-- All links get friction coefficients and as Gazebo don't read collors they specifeid again-->
+    <!-- All links get friction coefficients and visual materials for Gazebo Harmonic -->
     <gazebo reference="chassis_link">
-        <mu1> 0.2 </mu1>
-        <mu2> 0.2 </mu2>
-        <material>Gazebo/Grey</material>
+        <mu1>0.2</mu1>
+        <mu2>0.2</mu2>
+        <visual>
+            <material>
+                <ambient>0.5 0.5 0.5 1</ambient>
+                <diffuse>0.5 0.5 0.5 1</diffuse>
+                <specular>0.1 0.1 0.1 1</specular>
+            </material>
+        </visual>
     </gazebo>
     <gazebo reference="wheel_1_link">
-        <mu1> 0.2 </mu1>
-        <mu2> 0.2 </mu2>
-        <material>Gazebo/Black</material>
+        <mu1>0.8</mu1>
+        <mu2>0.8</mu2>
+        <visual>
+            <material>
+                <ambient>0.1 0.1 0.1 1</ambient>
+                <diffuse>0.1 0.1 0.1 1</diffuse>
+                <specular>0.1 0.1 0.1 1</specular>
+            </material>
+        </visual>
     </gazebo>
     <gazebo reference="wheel_2_link">
-        <mu1> 0.2 </mu1>
-        <mu2> 0.2 </mu2>
-        <material>Gazebo/Black</material>
+        <mu1>0.8</mu1>
+        <mu2>0.8</mu2>
+        <visual>
+            <material>
+                <ambient>0.1 0.1 0.1 1</ambient>
+                <diffuse>0.1 0.1 0.1 1</diffuse>
+                <specular>0.1 0.1 0.1 1</specular>
+            </material>
+        </visual>
     </gazebo>
     <gazebo reference="wheel_3_link">
-        <mu1> 0.2 </mu1>
-        <mu2> 0.2 </mu2>
-        <material>Gazebo/Black</material>
+        <mu1>0.8</mu1>
+        <mu2>0.8</mu2>
+        <visual>
+            <material>
+                <ambient>0.1 0.1 0.1 1</ambient>
+                <diffuse>0.1 0.1 0.1 1</diffuse>
+                <specular>0.1 0.1 0.1 1</specular>
+            </material>
+        </visual>
     </gazebo>
     <gazebo reference="wheel_4_link">
-        <mu1> 0.2 </mu1>
-        <mu2> 0.2 </mu2>
-        <material>Gazebo/Black</material>
+        <mu1>0.8</mu1>
+        <mu2>0.8</mu2>
+        <visual>
+            <material>
+                <ambient>0.1 0.1 0.1 1</ambient>
+                <diffuse>0.1 0.1 0.1 1</diffuse>
+                <specular>0.1 0.1 0.1 1</specular>
+            </material>
+        </visual>
     </gazebo>
     <gazebo reference="IMU_link">
-        <mu1> 0.2 </mu1>
-        <mu2> 0.2 </mu2>
-        <material>Gazebo/Red</material>
+        <mu1>0.2</mu1>
+        <mu2>0.2</mu2>
+        <visual>
+            <material>
+                <ambient>0.8 0.0 0.0 1</ambient>
+                <diffuse>0.8 0.0 0.0 1</diffuse>
+                <specular>0.1 0.1 0.1 1</specular>
+            </material>
+        </visual>
     </gazebo>
+    <!-- Gazebo Harmonic system plugins -->
     <gazebo>
-        <plugin name="joint_state_publisher" filename="libgazebo_ros_joint_state_publisher.so">
-            <jointName>wheel_1_joint,wheel_2_joint,wheel_3_joint,wheel_4_joint</jointName>
+        <!-- Joint State Publisher for Gazebo Harmonic -->
+        <plugin filename="gz-sim-joint-state-publisher-system" name="gz::sim::systems::JointStatePublisher">
+            <joint_name>wheel_1_joint</joint_name>
+            <joint_name>wheel_2_joint</joint_name>
+            <joint_name>wheel_3_joint</joint_name>
+            <joint_name>wheel_4_joint</joint_name>
+            <topic>joint_states</topic>
         </plugin>
     </gazebo>
@@ -43,30 +85,28 @@
 <!-- #################################################################################### -->
     <gazebo>
-        <!-- Gazebo plugin for differential drive -->
-        <plugin name="skid_steer_drive" filename="libgazebo_ros_diff_drive.so">
-            <ros>
-                <namespace> </namespace>
-            </ros>
-            <num_wheel_pairs>2</num_wheel_pairs>
-            <!-- Wheels 0 -->
+        <!-- Gazebo Harmonic differential drive plugin (skid-steer) -->
+        <plugin filename="gz-sim-diff-drive-system" name="gz::sim::systems::DiffDrive">
+            <!-- Wheels -->
             <left_joint>wheel_1_joint</left_joint>
+            <left_joint>wheel_4_joint</left_joint>
             <right_joint>wheel_2_joint</right_joint>
-            <!-- Wheels 1 -->
-            <left_joint>wheel_4_joint</left_joint>
             <right_joint>wheel_3_joint</right_joint>
             <!-- Kinematics -->
             <wheel_separation>${box_y+cyl_l}</wheel_separation>
-            <wheel_separation>${box_y+cyl_l}</wheel_separation>
-            <wheel_diameter>${cyl_r*2}</wheel_diameter>
-            <wheel_diameter>${cyl_r*2}</wheel_diameter>
+            <wheel_radius>${cyl_r}</wheel_radius>
             <!-- Limits -->
             <max_wheel_torque>1000</max_wheel_torque>
             <max_wheel_acceleration>5.0</max_wheel_acceleration>
-            <!-- Output -->
-            <publish_odom>false</publish_odom>
+            <!-- Topics -->
+            <topic>cmd_vel</topic>
+            <odom_topic>odom</odom_topic>
+            <tf_topic>tf</tf_topic>
+            <!-- Frames -->
+            <frame_id>odom</frame_id>
+            <child_frame_id>base_link</child_frame_id>
+            <!-- Output control -->
+            <publish_odom>true</publish_odom>
             <publish_odom_tf>false</publish_odom_tf>
             <publish_wheel_tf>false</publish_wheel_tf>
-            <!-- <odometry_frame>odom</odometry_frame> -->
-            <!-- <robot_base_frame>base_link</robot_base_frame> -->
         </plugin>
     </gazebo>

File: src/roburoc_description/urdf/VLP-16.urdf.xacro (robot description, xacro)
@@ -1,6 +1,6 @@
 <?xml version="1.0"?>
-<robot xmlns:xacro="http://www.ros.org/wiki/xacro" name="VLP-16">
+<robot xmlns:xacro="http://ros.org/wiki/xacro" name="VLP-16">
   <xacro:property name="M_PI" value="3.1415926535897931"/>
-  <xacro:macro name="VLP-16" params="*origin parent:=base_link name:=velodyne topic:=/velodyne_points hz:=10 lasers:=16 samples:=1875 collision_range:=0.3 min_range:=0.9 max_range:=130.0 noise:=0.008 min_angle:=-${M_PI} max_angle:=${M_PI} gpu:=false">
+  <xacro:macro name="VLP-16" params="*origin parent:=base_link name:=velodyne topic:=/velodyne_points hz:=10 lasers:=16 samples:=1875 collision_range:=0.3 min_range:=0.9 max_range:=130.0 noise:=0.008 min_angle:=-${M_PI} max_angle:=${M_PI} gpu:=true">
     <joint name="${name}_base_mount_joint" type="fixed">
       <xacro:insert_block name="origin"/>
@@ -50,98 +50,40 @@
       </visual>
     </link>
-    <!-- Gazebo requires the velodyne_gazebo_plugins package -->
+    <!-- Gazebo Harmonic GPU Lidar sensor -->
     <gazebo reference="${name}">
-      <xacro:if value="${gpu}">
-        <sensor type="gpu_ray" name="${name}-VLP16">
-          <pose>0 0 0 0 0 0</pose>
-          <visualize>false</visualize>
-          <update_rate>${hz}</update_rate>
-          <ray>
-            <scan>
-              <horizontal>
-                <samples>${samples}</samples>
-                <resolution>1</resolution>
-                <min_angle>${min_angle}</min_angle>
-                <max_angle>${max_angle}</max_angle>
-              </horizontal>
-              <vertical>
-                <samples>${lasers}</samples>
-                <resolution>1</resolution>
-                <min_angle>-${10.0*M_PI/180.0}</min_angle>
-                <max_angle>
-                  ${10.0*M_PI/180.0}</max_angle>
-              </vertical>
-            </scan>
-            <range>
-              <min>${collision_range}</min>
-              <max>${max_range+1}</max>
-              <resolution>0.001</resolution>
-            </range>
-            <noise>
-              <type>gaussian</type>
-              <mean>0.0</mean>
-              <stddev>0.0</stddev>
-            </noise>
-          </ray>
-          <!-- <plugin name="laser_controller" filename="libgazebo_ros_ray_sensor.so"> -->
-            <!-- <ros> -->
-              <!-- <argument>~/out:=scan</argument> -->
-            <!-- </ros> -->
-            <!-- <output_type>sensor_msgs/LaserScan</output_type> -->
-            <!-- <frame_name>${name}</frame_name> -->
-          <!-- </plugin> -->
-          <plugin name="gazebo_ros_laser_controller" filename="libgazebo_ros_velodyne_laser.so">
-            <ros>
-              <argument>~/out:=scan</argument>
-            </ros>
-            <topicName>${topic}</topicName>
-            <frameName>${name}</frameName>
-            <min_range>${min_range}</min_range>
-            <max_range>${max_range}</max_range>
-            <gaussianNoise>${noise}</gaussianNoise>
-          </plugin>
-        </sensor>
-      </xacro:if>
-      <xacro:unless value="${gpu}">
-        <sensor type="ray" name="${name}-VLP16">
-          <pose>0 0 0 0 0 0</pose>
-          <visualize>false</visualize>
-          <update_rate>${hz}</update_rate>
-          <ray>
-            <scan>
-              <horizontal>
-                <samples>${samples}</samples>
-                <resolution>1</resolution>
-                <min_angle>${min_angle}</min_angle>
-                <max_angle>${max_angle}</max_angle>
-              </horizontal>
-              <vertical>
-                <samples>${lasers}</samples>
-                <resolution>1</resolution>
-                <min_angle>-${10.0*M_PI/180.0}</min_angle>
-                <max_angle>
-                  ${10.0*M_PI/180.0}</max_angle>
-              </vertical>
-            </scan>
-            <range>
-              <min>${collision_range}</min>
-              <max>${max_range+1}</max>
-              <resolution>0.001</resolution>
-            </range>
-            <noise>
-              <type>gaussian</type>
-              <mean>0.0</mean>
-              <stddev>0.0</stddev>
-            </noise>
-          </ray>
-          <plugin name="gazebo_ros_laser_controller" filename="libgazebo_ros_velodyne_laser.so">
-            <topicName>${topic}</topicName>
-            <frameName>${name}</frameName>
-            <min_range>${min_range}</min_range>
-            <max_range>${max_range}</max_range>
-            <gaussianNoise>${noise}</gaussianNoise>
-          </plugin>
-        </sensor>
-      </xacro:unless>
+      <sensor name="${name}-VLP16" type="gpu_lidar">
+        <pose>0 0 0 0 0 0</pose>
+        <visualize>false</visualize>
+        <update_rate>${hz}</update_rate>
+        <always_on>true</always_on>
+        <topic>${topic}</topic>
+        <gz_frame_id>${name}</gz_frame_id>
+        <lidar>
+          <scan>
+            <horizontal>
+              <samples>${samples}</samples>
+              <resolution>1</resolution>
+              <min_angle>${min_angle}</min_angle>
+              <max_angle>${max_angle}</max_angle>
+            </horizontal>
+            <vertical>
+              <samples>${lasers}</samples>
+              <resolution>1</resolution>
+              <min_angle>-${15.0*M_PI/180.0}</min_angle>
+              <max_angle>${15.0*M_PI/180.0}</max_angle>
+            </vertical>
+          </scan>
+          <range>
+            <min>${min_range}</min>
+            <max>${max_range}</max>
+            <resolution>0.001</resolution>
+          </range>
+          <noise>
+            <type>gaussian</type>
+            <mean>0.0</mean>
+            <stddev>${noise}</stddev>
+          </noise>
+        </lidar>
+      </sensor>
     </gazebo>
   </xacro:macro>

File: src/roburoc_description/urdf/_d435.gazebo.xacro (robot description, xacro)
@@ -3,5 +3,6 @@
 License: Apache 2.0. See LICENSE file in root directory.
 Copyright(c) 2017 PAL Robotics, S.L. All Rights Reserved
-This is the Gazebo URDF model for the Intel RealSense D435 camera
+This is the Gazebo Harmonic URDF model for the Intel RealSense D435 camera
+Updated to use built-in rgbd_camera sensor with GPU acceleration
 -->
 <robot xmlns:xacro="http://ros.org/wiki/xacro">
@@ -14,14 +15,16 @@
       <kinematic>0</kinematic>
       <gravity>1</gravity>
-      <!--<mu>1</mu>-->
       <mu2>1</mu2>
       <fdir1>0 0 0</fdir1>
-      <!--<slip1>0</slip1>
-      <slip2>0</slip2>-->
       <kp>1e+13</kp>
       <kd>1</kd>
-      <!--<max_vel>0.01</max_vel>
-      <min_depth>0</min_depth>-->
-      <sensor name="${camera_name}color" type="camera">
+      <!-- Gazebo Harmonic RGBD Camera sensor with GPU acceleration -->
+      <sensor name="${camera_name}_rgbd" type="rgbd_camera">
+        <pose>0 0 0 0 0 0</pose>
+        <always_on>true</always_on>
+        <update_rate>30</update_rate>
+        <visualize>false</visualize>
+        <topic>${topics_ns}</topic>
+        <gz_frame_id>${color_optical_frame}</gz_frame_id>
         <camera name="${camera_name}">
           <horizontal_fov>${69.4*deg_to_rad}</horizontal_fov>
@@ -29,10 +32,16 @@
             <width>640</width>
             <height>480</height>
-            <format>RGB_INT8</format>
+            <format>R8G8B8</format>
           </image>
           <clip>
             <near>0.1</near>
-            <far>100</far>
+            <far>10.0</far>
           </clip>
+          <depth_camera>
+            <clip>
+              <near>0.2</near>
+              <far>10.0</far>
+            </clip>
+          </depth_camera>
           <noise>
             <type>gaussian</type>
@@ -41,99 +50,5 @@
           </noise>
         </camera>
-        <always_on>1</always_on>
-        <update_rate>30</update_rate>
-        <visualize>1</visualize>
       </sensor>
-      <sensor name="${camera_name}ired1" type="camera">
-        <camera name="${camera_name}">
-          <horizontal_fov>${85.2*deg_to_rad}</horizontal_fov>
-          <image>
-            <width>1280</width>
-            <height>720</height>
-            <format>L_INT8</format>
-          </image>
-          <clip>
-            <near>0.1</near>
-            <far>100</far>
-          </clip>
-          <noise>
-            <type>gaussian</type>
-            <mean>0.0</mean>
-            <stddev>0.05</stddev>
-          </noise>
-        </camera>
-        <always_on>1</always_on>
-        <update_rate>90</update_rate>
-        <visualize>0</visualize>
-      </sensor>
-      <sensor name="${camera_name}ired2" type="camera">
-        <camera name="${camera_name}">
-          <horizontal_fov>${85.2*deg_to_rad}</horizontal_fov>
-          <image>
-            <width>1280</width>
-            <height>720</height>
-            <format>L_INT8</format>
-          </image>
-          <clip>
-            <near>0.1</near>
-            <far>100</far>
-          </clip>
-          <noise>
-            <type>gaussian</type>
-            <mean>0.0</mean>
-            <stddev>0.05</stddev>
-          </noise>
-        </camera>
-        <always_on>1</always_on>
-        <update_rate>90</update_rate>
-        <visualize>0</visualize>
-      </sensor>
-      <sensor name="${camera_name}depth" type="depth">
-        <camera name="${camera_name}">
-          <horizontal_fov>${85.2*deg_to_rad}</horizontal_fov>
-          <image>
-            <width>1280</width>
-            <height>720</height>
-          </image>
-          <clip>
-            <near>0.1</near>
-            <far>100</far>
-          </clip>
-          <noise>
-            <type>gaussian</type>
-            <mean>0.0</mean>
-            <stddev>0.100</stddev>
-          </noise>
-        </camera>
-        <always_on>1</always_on>
-        <update_rate>90</update_rate>
-        <visualize>0</visualize>
-      </sensor>
-    </gazebo>
-    <gazebo>
-      <plugin name="${topics_ns}" filename="librealsense_gazebo_plugin.so">
-        <prefix>${camera_name}</prefix>
-        <depthUpdateRate>30.0</depthUpdateRate>
-        <colorUpdateRate>30.0</colorUpdateRate>
-        <infraredUpdateRate>30.0</infraredUpdateRate>
-        <depthTopicName>${topics_ns}/depth/image_raw</depthTopicName>
-        <depthCameraInfoTopicName>${topics_ns}/depth/camera_info</depthCameraInfoTopicName>
-        <colorTopicName>${topics_ns}/color/image_raw</colorTopicName>
-        <colorCameraInfoTopicName>${topics_ns}/color/camera_info</colorCameraInfoTopicName>
-        <infrared1TopicName>${topics_ns}/infra1/image_raw</infrared1TopicName>
-        <infrared1CameraInfoTopicName>${topics_ns}/infra1/camera_info</infrared1CameraInfoTopicName>
-        <infrared2TopicName>${topics_ns}/infra2/image_raw</infrared2TopicName>
-        <infrared2CameraInfoTopicName>${topics_ns}/infra2/camera_info</infrared2CameraInfoTopicName>
-        <colorOpticalframeName>${color_optical_frame}</colorOpticalframeName>
-        <depthOpticalframeName>${depth_optical_frame}</depthOpticalframeName>
-        <infrared1OpticalframeName>${infrared1_optical_frame}</infrared1OpticalframeName>
-        <infrared2OpticalframeName>${infrared2_optical_frame}</infrared2OpticalframeName>
-        <rangeMinDepth>0.2</rangeMinDepth>
-        <rangeMaxDepth>10.0</rangeMaxDepth>
-        <pointCloud>${publish_pointcloud}</pointCloud>
-        <pointCloudTopicName>${topics_ns}/depth/color/points</pointCloudTopicName>
-        <pointCloudCutoff>0.25</pointCloudCutoff>
-        <pointCloudCutoffMax>9.0</pointCloudCutoffMax>
-      </plugin>
     </gazebo>
   </xacro:macro>
