Commit message: Reorganize robot URDF/XACRO structure, add new sensor definitions

File: src/roburoc_description/urdf/base/chassis_and_wheels.xacro (robot description, xacro)
@@ -1,10 +1,31 @@
 <?xml version="1.0"?>
-<robot xmlns:xacro="http://www.ros.org/wiki/xacro"  name="RobuROC">
-    <!-- This is RobuROC model for rviz visualisation -->
-    <!-- Model visualisation is made of stl files and collison is made of simple shapes box and cylinders-->
+<!--
+  chassis_and_wheels.xacro - RobuROC Base Platform
+  This file defines the core robot structure:
+    - base_link: Empty root link (ROS convention)
+    - base_footprint: Ground-level link for SLAM
+    - chassis_link: Main robot body with STL mesh
+    - wheel_1-4_links: Four wheels (continuous joints)
+  Coordinate frame:
+    - X: Forward
+    - Y: Left
+    - Z: Up
+  Wheel numbering (top view):
+    1 (+x,+y) ---- 2 (+x,-y)
+        |   FRONT   |
+        |           |
+    4 (-x,+y) ---- 3 (-x,-y)
+  Dependencies:
+    - common/properties.xacro (dimensions)
+    - common/materials.xacro (colors)
+    - common/inertia_macros.xacro (inertia calculations)
+-->
+<robot xmlns:xacro="http://www.ros.org/wiki/xacro" name="RobuROC">
     <!-- Initial link is empty link called base_link -->
     <link name="base_link"></link>
-    <!-- BASE_FOOTPRINT LINK -->
-    <!-- link for SLAM -->
+    <!-- ############################################## -->
+    <!--              BASE_FOOTPRINT LINK              -->
+    <!-- ############################################## -->
+    <!-- Ground-level link for SLAM algorithms -->
     <joint name="base_footprint_joint" type="fixed">
         <parent link="base_link"/>
@@ -14,8 +35,7 @@
     <link name="base_footprint">
     </link>
-    <!-- ##############################################  -->
-    <!--                Chassis Link                     -->
-    <!-- ##############################################  -->
-    <!-- Chassis joint has been off seted in z axis and set to fixed-->
+    <!-- ############################################## -->
+    <!--                Chassis Link                   -->
+    <!-- ############################################## -->
     <joint name="chassis_joint" type="fixed">
         <parent link="base_link"/>
@@ -40,7 +60,7 @@
         </xacro:inertial_box>
     </link>
-    <!-- ##############################################  -->
-    <!--                WHEEL 1  +x +y                   -->
-    <!-- ##############################################  -->
+    <!-- ############################################## -->
+    <!--                WHEEL 1  +x +y                 -->
+    <!-- ############################################## -->
     <joint name="wheel_1_joint" type="continuous">
         <origin xyz="${wheel_1_origin}" rpy="${-rot_90} 0 0"/>
@@ -69,7 +89,7 @@
         </xacro:inertial_cylinder>
     </link>
-    <!-- ##############################################  -->
-    <!--                WHEEL 2  +x -y                   -->
-    <!-- ##############################################  -->
+    <!-- ############################################## -->
+    <!--                WHEEL 2  +x -y                 -->
+    <!-- ############################################## -->
     <joint name="wheel_2_joint" type="continuous">
         <origin xyz="${wheel_2_origin}" rpy="${-rot_90} 0 0"/>
@@ -98,7 +118,7 @@
         </xacro:inertial_cylinder>
     </link>
-    <!-- ##############################################  -->
-    <!--                WHEEL 3  -x -y                   -->
-    <!-- ##############################################  -->
+    <!-- ############################################## -->
+    <!--                WHEEL 3  -x -y                 -->
+    <!-- ############################################## -->
     <joint name="wheel_3_joint" type="continuous">
         <origin xyz="${wheel_3_origin}" rpy="${-rot_90} 0 0"/>
@@ -127,7 +147,7 @@
         </xacro:inertial_cylinder>
     </link>
-    <!-- ##############################################  -->
-    <!--                WHEEL 4  -x +y                   -->
-    <!-- ##############################################  -->
+    <!-- ############################################## -->
+    <!--                WHEEL 4  -x +y                 -->
+    <!-- ############################################## -->
     <joint name="wheel_4_joint" type="continuous">
         <origin xyz="${wheel_4_origin}" rpy="${-rot_90} 0 0"/>

File: src/roburoc_description/urdf/common/properties.xacro (robot description, xacro)
@@ -1,5 +1,17 @@
 <?xml version="1.0"?>
-<robot xmlns:xacro="http://www.ros.org/wiki/xacro" >
-    <!-- This file is not a robot in and of itself, it just contains some useful tags that could be included in any robot -->
+<!--
+  properties.xacro - RobuROC Robot Properties
+  This file contains all dimensional properties and position parameters
+  for the RobuROC robot. It is included by all other xacro files that
+  need access to robot dimensions.
+  Contents:
+    - Chassis dimensions (box_x, box_y, box_z, etc.)
+    - Wheel dimensions and positions
+    - Camera mounting positions
+    - Lidar mounting position
+    - STL scale factor
+  Include hierarchy: This is the first file included by roburoc.urdf.xacro
+-->
+<robot xmlns:xacro="http://www.ros.org/wiki/xacro">
     <!-- ######################################### -->
     <!--                Chassis                    -->
@@ -40,8 +52,6 @@
     <xacro:property name="camera_1_origin" value="${camera_off_x} 0 ${camera_off_z}" />
     <xacro:property name="camera_2_origin" value="${-camera_off_x} 0 ${camera_off_z}" />
-    <!-- <xacro:property name="camera_2_origin" value="${camera_off_x-0.05} -0.32 ${camera_off_z}" /> -->
     <xacro:property name="camera_1_rotation" value="0 ${(camera_rot)*pi/180} 0" />
     <xacro:property name="camera_2_rotation" value="0 ${(camera_rot-2)*pi/180} ${pi}" />
-    <!-- <xacro:property name="camera_2_rotation" value="0 ${camera_rot} 0" /> -->
     <!-- ######################################### -->
     <!--                    Lidar                  -->
@@ -50,54 +60,3 @@
     <xacro:property name="lidar_off_z" value="${box_off_z+0.155}" />
     <xacro:property name="lidar_origin" value="${lidar_off_x} 0 ${lidar_off_z}" />
-    <!-- Specify some colours -->
-    <material name="white">
-        <color rgba="1 1 1 1"/>
-    </material>
-    <material name="orange">
-        <color rgba="1 0.3 0.1 1"/>
-    </material>
-    <material name="blue">
-        <color rgba="0.2 0.2 1 1"/>
-    </material>
-    <material name="green">
-        <color rgba="0.2 1 0.2 1"/>
-    </material>
-    <material name="red">
-        <color rgba="1 0.2 0.2 1"/>
-    </material>
-    <material name="black">
-        <color rgba="0 0 0 1"/>
-    </material>
-    <material name="grey">
-        <color rgba="0.5 0.5 0.5 1"/>
-    </material>
-    <!-- Specify some standard inertial calculations https://en.wikipedia.org/wiki/List_of_moments_of_inertia -->
-    <!-- These make use of xacro's mathematical functionality -->
-    <xacro:macro name="inertial_sphere" params="mass radius *origin">
-        <inertial>
-            <xacro:insert_block name="origin"/>
-            <mass value="${mass}" />
-            <inertia ixx="${(2/5) * mass * (radius*radius)}" ixy="0.0" ixz="0.0"
-                    iyy="${(2/5) * mass * (radius*radius)}" iyz="0.0"
-                    izz="${(2/5) * mass * (radius*radius)}" />
-        </inertial>
-    </xacro:macro>
-    <xacro:macro name="inertial_box" params="mass x y z *origin">
-        <inertial>
-            <xacro:insert_block name="origin"/>
-            <mass value="${mass}" />
-            <inertia ixx="${(1/12) * mass * (y*y+z*z)}" ixy="0.0" ixz="0.0"
-                    iyy="${(1/12) * mass * (x*x+z*z)}" iyz="0.0"
-                    izz="${(1/12) * mass * (x*x+y*y)}" />
-        </inertial>
-    </xacro:macro>
-    <xacro:macro name="inertial_cylinder" params="mass length radius *origin">
-        <inertial>
-            <xacro:insert_block name="origin"/>
-            <mass value="${mass}" />
-            <inertia ixx="${(1/12) * mass * (3*radius*radius + length*length)}" ixy="0.0" ixz="0.0"
-                    iyy="${(1/12) * mass * (3*radius*radius + length*length)}" iyz="0.0"
-                    izz="${(1/2) * mass * (radius*radius)}" />
-        </inertial>
-    </xacro:macro>
 </robot>

File: src/roburoc_description/urdf/gazebo/simulation.xacro (robot description, xacro)
@@ -1,7 +1,25 @@
 <?xml version="1.0"?>
+<!--
+  simulation.xacro - Gazebo Harmonic Simulation Configuration
+  This file configures Gazebo-specific properties for the robot:
+    - Friction coefficients (mu1, mu2) for physics simulation
+    - Visual materials for Gazebo rendering
+    - Joint state publisher plugin
+    - Differential drive plugin (skid-steer configuration)
+  Note: This file does NOT include sensor simulation - those are
+  defined alongside their respective sensors in the sensors/ directory.
+  Plugins:
+    - gz-sim-joint-state-publisher-system: Publishes wheel joint states
+    - gz-sim-diff-drive-system: Skid-steer drive controller
+  Topics:
+    - /joint_states: Wheel positions
+    - /cmd_vel: Velocity commands (input)
+    - /odom: Odometry (output)
+-->
 <robot xmlns:xacro="http://www.ros.org/wiki/xacro">
-    <!-- This is RobuROC model for Gazebo Harmonic simulation -->
-    <!-- Model visualisation and collision is made of simple shapes box and cylinders-->
-    <!-- All links get friction coefficients and visual materials for Gazebo Harmonic -->
+    <!-- ############################################## -->
+    <!--              Link Friction/Materials          -->
+    <!-- ############################################## -->
+    <!-- Chassis: Low friction (slides if pushed) -->
     <gazebo reference="chassis_link">
         <mu1>0.2</mu1>
@@ -15,4 +33,5 @@
         </visual>
     </gazebo>
+    <!-- Wheels: High friction for traction -->
     <gazebo reference="wheel_1_link">
         <mu1>0.8</mu1>
@@ -59,4 +78,5 @@
         </visual>
     </gazebo>
+    <!-- IMU: Low friction, red visual -->
     <gazebo reference="IMU_link">
         <mu1>0.2</mu1>
@@ -70,7 +90,9 @@
         </visual>
     </gazebo>
-    <!-- Gazebo Harmonic system plugins -->
+    <!-- ############################################## -->
+    <!--              System Plugins                   -->
+    <!-- ############################################## -->
+    <!-- Joint State Publisher -->
     <gazebo>
-        <!-- Joint State Publisher for Gazebo Harmonic -->
         <plugin filename="gz-sim-joint-state-publisher-system" name="gz::sim::systems::JointStatePublisher">
             <joint_name>wheel_1_joint</joint_name>
@@ -81,11 +103,10 @@
         </plugin>
     </gazebo>
-<!-- #################################################################################### -->
-<!--                                Differential drive                                    -->
-<!-- #################################################################################### -->
+    <!-- ############################################## -->
+    <!--           Differential Drive (Skid-Steer)     -->
+    <!-- ############################################## -->
     <gazebo>
-        <!-- Gazebo Harmonic differential drive plugin (skid-steer) -->
         <plugin filename="gz-sim-diff-drive-system" name="gz::sim::systems::DiffDrive">
-            <!-- Wheels -->
+            <!-- Wheel configuration (skid-steer: 2 left, 2 right) -->
             <left_joint>wheel_1_joint</left_joint>
             <left_joint>wheel_4_joint</left_joint>

Commit message: Add IMU sensor support with joint and plugin configurations for Gazebo simulation

File: src/roburoc_description/urdf/base/chassis_and_wheels.xacro (robot description, xacro)
@@ -36,4 +36,27 @@
     </link>
     <!-- ############################################## -->
+    <!--                  IMU Link                     -->
+    <!-- ############################################## -->
+    <!-- IMU sensor mounted on chassis -->
+    <joint name="imu_joint" type="fixed">
+        <parent link="base_link"/>
+        <child link="IMU_link"/>
+        <origin xyz="0 0 0.1" rpy="0 0 0"/>
+    </joint>
+    <link name="IMU_link">
+        <visual>
+            <geometry>
+                <box size="0.02 0.02 0.01"/>
+            </geometry>
+            <material name="red">
+                <color rgba="0.8 0 0 1"/>
+            </material>
+        </visual>
+        <inertial>
+            <mass value="0.01"/>
+            <inertia ixx="0.0001" ixy="0" ixz="0" iyy="0.0001" iyz="0" izz="0.0001"/>
+        </inertial>
+    </link>
+    <!-- ############################################## -->
     <!--                Chassis Link                   -->
     <!-- ############################################## -->

File: src/roburoc_description/urdf/gazebo/simulation.xacro (robot description, xacro)
@@ -93,4 +93,9 @@
     <!--              System Plugins                   -->
     <!-- ############################################## -->
+    <!-- IMU System Plugin (required for IMU sensor) -->
+    <gazebo>
+        <plugin filename="gz-sim-imu-system" name="gz::sim::systems::Imu">
+        </plugin>
+    </gazebo>
     <!-- Joint State Publisher -->
     <gazebo>
@@ -134,3 +139,87 @@
         </plugin>
     </gazebo>
+    <!-- ############################################## -->
+    <!--              IMU Sensor Plugin                -->
+    <!-- ############################################## -->
+    <gazebo reference="IMU_link">
+        <sensor name="imu_sensor" type="imu">
+            <always_on>1</always_on>
+            <update_rate>100</update_rate>
+            <topic>imu</topic>
+            <gz_frame_id>IMU_link</gz_frame_id>
+            <imu>
+                <enable_orientation>1</enable_orientation>
+                <angular_velocity>
+                    <x>
+                        <noise type="gaussian">
+                            <mean>0</mean>
+                            <stddev>0.009</stddev>
+                            <bias_mean>0.00075</bias_mean>
+                            <bias_stddev>0.005</bias_stddev>
+                            <dynamic_bias_stddev>0.00002</dynamic_bias_stddev>
+                            <dynamic_bias_correlation_time>400.0</dynamic_bias_correlation_time>
+                            <precision>0.00025</precision>
+                        </noise>
+                    </x>
+                    <y>
+                        <noise type="gaussian">
+                            <mean>0</mean>
+                            <stddev>0.009</stddev>
+                            <bias_mean>0.00075</bias_mean>
+                            <bias_stddev>0.005</bias_stddev>
+                            <dynamic_bias_stddev>0.00002</dynamic_bias_stddev>
+                            <dynamic_bias_correlation_time>400.0</dynamic_bias_correlation_time>
+                            <precision>0.00025</precision>
+                        </noise>
+                    </y>
+                    <z>
+                        <noise type="gaussian">
+                            <mean>0</mean>
+                            <stddev>0.009</stddev>
+                            <bias_mean>0.00075</bias_mean>
+                            <bias_stddev>0.005</bias_stddev>
+                            <dynamic_bias_stddev>0.00002</dynamic_bias_stddev>
+                            <dynamic_bias_correlation_time>400.0</dynamic_bias_correlation_time>
+                            <precision>0.00025</precision>
+                        </noise>
+                    </z>
+                </angular_velocity>
+                <linear_acceleration>
+                    <x>
+                        <noise type="gaussian">
+                            <mean>0</mean>
+                            <stddev>0.021</stddev>
+                            <bias_mean>0.05</bias_mean>
+                            <bias_stddev>0.0075</bias_stddev>
+                            <dynamic_bias_stddev>0.000375</dynamic_bias_stddev>
+                            <dynamic_bias_correlation_time>175.0</dynamic_bias_correlation_time>
+                            <precision>0.005</precision>
+                        </noise>
+                    </x>
+                    <y>
+                        <noise type="gaussian">
+                            <mean>0</mean>
+                            <stddev>0.021</stddev>
+                            <bias_mean>0.05</bias_mean>
+                            <bias_stddev>0.0075</bias_stddev>
+                            <dynamic_bias_stddev>0.000375</dynamic_bias_stddev>
+                            <dynamic_bias_correlation_time>175.0</dynamic_bias_correlation_time>
+                            <precision>0.005</precision>
+                        </noise>
+                    </y>
+                    <z>
+                        <noise type="gaussian">
+                            <mean>0</mean>
+                            <stddev>0.021</stddev>
+                            <bias_mean>0.05</bias_mean>
+                            <bias_stddev>0.0075</bias_stddev>
+                            <dynamic_bias_stddev>0.000375</dynamic_bias_stddev>
+                            <dynamic_bias_correlation_time>175.0</dynamic_bias_correlation_time>
+                            <precision>0.005</precision>
+                        </noise>
+                    </z>
+                </linear_acceleration>
+            </imu>
+        </sensor>
+    </gazebo>
 </robot>
