Commit message: fix: update joint origin parameters for livox_mid360_rtk sensor configuration

File: src/roburoc_description/urdf/sensors/livox_mid360_rtk.urdf.xacro (robot description, xacro)
@@ -28,5 +28,5 @@
         <parent link="base_link"/>
         <child  link="livox_frame"/>
-        <origin xyz="0.6625 0.0 0.645" rpy="0 0.39373590 0"/>
+        <origin xyz="0.6625 0.0 0.7625" rpy="0 0.44457789 0"/>
     </joint>
     <!-- ── u-blox ZED-F9P RTK antenna ───────────────────────────────────── -->

Commit message: fix: slight changes to sensor extrinsics, renamed gps to gps_link

File: src/roburoc_description/urdf/sensors/livox_mid360_rtk.urdf.xacro (robot description, xacro)
@@ -6,13 +6,17 @@
     - u-blox ZED-F9P RTK-GPS receiver
   Frames contributed to the TF tree:
-    livox_frame  — MID360 sensor origin.  Matches the livox_ros_driver2 default
-                   frame_id ("livox_frame") so no extra static TF is needed.
-                   FAST-LIO2 anchors its "body" frame here.
-    gps          — RTK antenna phase centre.  Matches the ublox_gps node default
-                   output frame_id ("gps") so NavSatFix messages are referenced correctly.
+    livox_frame      — MID360 sensor origin.  Matches the livox_ros_driver2 default
+                       frame_id ("livox_frame") so no extra static TF is needed.
+                       FAST-LIO2 calls this frame "body" internally.
+    gps_link — RTK antenna phase centre.  Physical attachment frame; uses the
+                       _link suffix convention (REP-105).  The ublox driver stamps its
+                       NavSatFix messages with frame_id="gps" (driver default).
   All transforms are measured from the base_link origin (ground plane centred
   between the four wheel contact patches, X forward, Y left, Z up per REP-105).
   No visual or collision geometry is defined: this configuration is intended for
   real hardware only, not simulation.
+  TF tree (from this file):
+    base_link → livox_frame
+    base_link → gps_link
   See also:
     launch/sensors/livox_mid360_rtk.launch.py   — drivers for this config
@@ -28,5 +32,5 @@
         <parent link="base_link"/>
         <child  link="livox_frame"/>
-        <origin xyz="0.6625 0.0 0.7625" rpy="0 0.44457789 0"/>
+        <origin xyz="0.60 0.0 0.7625" rpy="0 0.44457789 0"/>
     </joint>
     <!-- ── u-blox ZED-F9P RTK antenna ───────────────────────────────────── -->
@@ -34,9 +38,12 @@
     <!-- 180° (yaw = π) because the connector faces forward on the mount.    -->
     <!-- Measurements: x=-0.428 m, y=0.295 m (left of centre), z=1.495 m.   -->
-    <link name="gps"/>
+    <!-- Note: the ublox driver publishes NavSatFix with frame_id="gps"      -->
+    <!-- (driver default); that bare name is left as-is.  This URDF link uses the -->
+    <!-- _link suffix convention for physical attachment frames.              -->
+    <link name="gps_link"/>
     <joint name="gps_joint" type="fixed">
         <parent link="base_link"/>
-        <child  link="gps"/>
-        <origin xyz="-0.428 0.295 1.495" rpy="0 0 3.14159265"/>
+        <child  link="gps_link"/>
+        <origin xyz="-0.4775 0.285 1.495" rpy="0 0 3.14159265"/>
     </joint>
 </robot>

Commit message: feat: tuning and debugging WIP

File: src/roburoc_description/urdf/sensors/livox_mid360_rtk.urdf.xacro (robot description, xacro)
@@ -32,5 +32,5 @@
         <parent link="base_link"/>
         <child  link="livox_frame"/>
-        <origin xyz="0.60 0.0 0.7625" rpy="0 0.44457789 0"/>
+        <origin xyz="0.60 0.0 0.7625" rpy="0 0.43618904 0"/>
     </joint>
     <!-- ── u-blox ZED-F9P RTK antenna ───────────────────────────────────── -->
